Commit message: added my_rb1_robot

File: my_rb1_description/urdf/my_rb1_robot.urdf (robot description, URDF)
Before this commit: robot robot, 6 links, 5 joints
Links:
- removed link link_chassis
- removed link link_laser_scan
- removed link link_left_front_wheel
- removed link link_left_rear_wheel
- removed link link_right_front_wheel
- removed link link_right_rear_wheel
- added link base_link, mass ${base_mass}; collision cylinder length=0.3 radius=0.25; visual cylinder length=0.3 radius=0.25
- added link front_caster, mass 1; collision sphere radius=0.025; visual sphere radius=0.025
- added link front_laser, mass 1; collision cylinder length=0.10 radius=0.075; visual cylinder length=0.10 radius=0.075
- added link left_wheel, mass 1; collision cylinder length=0.03 radius=0.05; visual cylinder length=0.03 radius=0.05
- added link rear_caster, mass 1; collision sphere radius=0.025; visual sphere radius=0.025
- added link right_wheel, mass 1; collision cylinder length=0.03 radius=0.05; visual cylinder length=0.03 radius=0.05
Joints:
- removed joint joint_chassis_left_front_wheel
- removed joint joint_chassis_left_rear_wheel
- removed joint joint_chassis_right_front_wheel
- removed joint joint_chassis_right_rear_wheel
- removed joint joint_laser_scan_chassis
- added joint joint_base_front_caster: type fixed, parent base_link, child front_caster, origin xyz=-0.1 0.0 -0.15 rpy=0 0 0, axis 1 0 0, limit effort=10000 velocity=1000
- added joint joint_base_left_wheel: type continuous, parent base_link, child left_wheel, origin xyz=0 -0.2 -0.15 rpy=0 0 0, axis 0 1 0, limit effort=10000 velocity=1000
- added joint joint_base_rear_caster: type fixed, parent base_link, child rear_caster, origin xyz=0.1 0.0 -0.15 rpy=0 0 0, axis 1 0 0, limit effort=10000 velocity=1000
- added joint joint_base_right_wheel: type continuous, parent base_link, child right_wheel, origin xyz=0 0.2 -0.15 rpy=0 0 0, axis 0 1 0, limit effort=10000 velocity=1000
- added joint joint_front_laser: type fixed, parent base_link, child front_laser, origin xyz=0.25 0 0.075 rpy=${pi} 0 0

Commit message: Running Robot in Gazebo no problem

File: my_rb1_description/urdf/my_rb1_robot.urdf (robot description, URDF)
Before this commit: robot my_rb1_robot, 6 links, 5 joints
Links:
- added link link_footprint, mass 0
- link left_wheel: geometry collision cylinder length=0.03 radius=0.025; visual cylinder length=0.03 radius=0.025
- link right_wheel: geometry collision cylinder length=0.03 radius=0.025; visual cylinder length=0.03 radius=0.025
Joints:
- added joint joint_base_link_footprint: type fixed, parent link_footprint, child base_link, origin xyz=0 0 0 rpy=0 0 0, axis 0 0 0, limit effort=10000 velocity=1000

File: my_rb1_description/urdf/my_rb1_robot.xacro (robot description, xacro)
@@ -1,4 +1,5 @@
 <?xml version="1.0" ?>
 <robot name="my_rb1_robot" xmlns:xacro="http://www.ros.org/wiki/xacro">
+    <xacro:include filename="$(find my_rb1_description)/urdf/my_rb1_robot.gazebo" />
     <!-- Parameters -->
     <xacro:property name="base_mass" value="22" />

Commit message: RVIZ working Good

File: my_rb1_description/urdf/my_rb1_robot.urdf (robot description, URDF)
Before this commit: robot my_rb1_robot, 6 links, 5 joints
Links:
- added link link_footprint; visual box size=0.01 0.01 0
Joints:
- added joint joint_base_footprint: type planar, parent link_footprint, child base_link, origin xyz=0 0 0 rpy=0 0 0
- joint joint_base_front_caster: origin xyz=-0.1 0.0 -0.15 rpy=0 0 0 -> xyz=0.1 0.0 -0.15 rpy=0 0 0
- joint joint_base_left_wheel: origin xyz=0 -0.2 -0.15 rpy=0 0 0 -> xyz=0 0.2 -0.15 rpy=0 0 0
- joint joint_base_rear_caster: origin xyz=0.1 0.0 -0.15 rpy=0 0 0 -> xyz=-0.1 0.0 -0.15 rpy=0 0 0
- joint joint_base_right_wheel: origin xyz=0 0.2 -0.15 rpy=0 0 0 -> xyz=0 -0.2 -0.15 rpy=0 0 0

File: my_rb1_description/urdf/my_rb1_robot.xacro (robot description, xacro)
@@ -4,4 +4,4 @@
     <xacro:property name="base_mass" value="22" />
     <xacro:property name="pi" value="3.1415926535897931"/>
-    <xacro:include filename="$(find my_rb1_description)/urdf/my_rb1_robot.urdf" />
-    </robot>
+    <xacro:include filename="$(find my_rb1_description)/urdf/my_rb1_robot.urdf"/>
+</robot>

Commit message: Gazebo working goood

File: my_rb1_description/urdf/my_rb1_robot.urdf (robot description, URDF)
Before this commit: robot my_rb1_robot, 7 links, 6 joints
Links:
- link link_footprint: mass 0 -> None; geometry visual box size=0.1 0.1 0
Joints:
- joint joint_base_front_caster: origin xyz=-0.1 0.0 -0.15 rpy=0 0 0 -> xyz=0.1 0.0 -0.15 rpy=0 0 0
- joint joint_base_left_wheel: origin xyz=0 -0.2 -0.15 rpy=0 0 0 -> xyz=0 0.2 -0.15 rpy=0 0 0
- joint joint_base_rear_caster: origin xyz=0.1 0.0 -0.15 rpy=0 0 0 -> xyz=-0.1 0.0 -0.15 rpy=0 0 0
- joint joint_base_right_wheel: origin xyz=0 0.2 -0.15 rpy=0 0 0 -> xyz=0 -0.2 -0.15 rpy=0 0 0

Commit message: Gazebo working Good

File: my_rb1_description/urdf/my_rb1_robot.urdf (robot description, URDF)
Before this commit: robot my_rb1_robot, 7 links, 6 joints
Links:
- removed link rear_caster
- added link back_caster, mass 1; collision sphere radius=0.025; visual sphere radius=0.025
Joints:
- joint joint_base_rear_caster: child rear_caster -> back_caster

Commit message: review

File: my_rb1_description/urdf/my_rb1_robot.urdf (robot description, URDF)
Before this commit: robot my_rb1_robot, 7 links, 6 joints
Links:
- link link_footprint: geometry visual box size=0.01 0.01 0
Joints:
- removed joint joint_base_link_footprint
- added joint joint_base_footprint: type planar, parent link_footprint, child base_link, origin xyz=0 0 0.15 rpy=0 0 0

Commit message: review

File: my_rb1_description/urdf/my_rb1_robot.urdf (robot description, URDF)
Before this commit: robot my_rb1_robot, 7 links, 6 joints
Links:
- link link_footprint: geometry visual box size=0.1 0.1 0
Joints:
- joint joint_base_footprint: axis (none) -> 0 0 0; limit (none) -> effort=10000 velocity=1000; origin xyz=0 0 0.15 rpy=0 0 0 -> xyz=0 0 0 rpy=0 0 -0.15; type planar -> fixed

Commit message: Robot without iddle motion

File: my_rb1_description/urdf/my_rb1_robot.urdf (robot description, URDF)
Before this commit: robot my_rb1_robot, 7 links, 6 joints
Joints:
- joint joint_base_footprint: origin xyz=0 0 0 rpy=0 0 -0.15 -> xyz=0 0 0 rpy=0 0 0

Commit message: TF foot print fixed

File: my_rb1_description/urdf/my_rb1_robot.urdf (robot description, URDF)
Before this commit: robot my_rb1_robot, 7 links, 6 joints
Links:
- link link_footprint: geometry visual box size=0.01 0.01 0
Joints:
- joint joint_base_footprint: origin xyz=0 0 0 rpy=0 0 0 -> xyz=0 0 0.15 rpy=0 0 0
